Commit message: feat: :sparkles: Add first part and second part of the challenge
Add simulation, localisation, classes and setup file

File: urdf/puzzlebot_jetson_ed_urdf.urdf (robot description, URDF)
Before this commit: robot Puzzlebot Jetson-Lidar Ed., 2 links, 1 joints
Links:
- link chassis: geometry collision mesh filename=package://puzzlebot_localisation/models/MCR2_1000_13_Chassi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; visual mesh filename=package://puzzlebot_localisation/models/MCR2_1000_13_Chassi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

Commit message: feat: :sparkles: Added broadcast file for doing the tf

File: urdf/puzzlebot_jetson_ed_urdf.urdf (robot description, URDF)
Before this commit: robot Puzzlebot Jetson-Lidar Ed., 2 links, 1 joints
Links:
- added link wl_link; visual mesh filename=package://puzzlebot_localisation/models/MCR2_1000_1_1_Wheel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
- added link wr_link; visual mesh filename=package://puzzlebot_localisation/models/MCR2_1000_1_1_Wheel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
Joints:
- added joint left_wheel: type continuous, parent chassis, child wl_link, origin xyz=0 0 0, axis 0 0 1
- added joint right_wheel: type continuous, parent chassis, child wr_link, origin xyz=0 0 0, axis 0 0 1

Commit message: fix: :ambulance: Rollback the urdf file and add rviz config

File: urdf/puzzlebot_jetson_ed_urdf.urdf (robot description, URDF)
Before this commit: robot Puzzlebot Jetson-Lidar Ed., 4 links, 3 joints
Links:
- removed link wl_link
- removed link wr_link
Joints:
- removed joint left_wheel
- removed joint right_wheel

Commit message: feat: :sparkles: Add transform between odom and base link, also set odom as the inertial frame

File: urdf/puzzlebot_jetson_ed_urdf.urdf (robot description, URDF)
Before this commit: robot Puzzlebot Jetson-Lidar Ed., 2 links, 1 joints
Links:
- added link wl_link; visual mesh filename=package://puzzlebot_localisation/models/MCR2_1000_1_1_Wheel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
- added link wr_link; visual mesh filename=package://puzzlebot_localisation/models/MCR2_1000_1_1_Wheel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
Joints:
- added joint leftWheel: type continuous, parent chassis, child wl_link, origin xyz=0 0 0, axis 0 0 1
- added joint rightWheel: type continuous, parent chassis, child wr_link, origin xyz=0 0 0, axis 0 0 1

Commit message: fix: :bug: Fixed quaternions for orientation in odom and transformation

File: urdf/puzzlebot_jetson_ed_urdf.urdf (robot description, URDF)
Before this commit: robot Puzzlebot Jetson-Lidar Ed., 4 links, 3 joints
Joints:
- joint leftWheel: axis 0 0 1 -> (none); origin xyz=0 0 0 -> xyz=0.0 0.0 0.0
- joint rightWheel: axis 0 0 1 -> (none); origin xyz=0 0 0 -> xyz=0.0 0.0 0.0

Commit message: feat: :sparkles: Added dictionary for trajectories and added color and collisions to urdf model

File: urdf/puzzlebot_jetson_ed_urdf.urdf (robot description, URDF)
Before this commit: robot Puzzlebot Jetson-Lidar Ed., 4 links, 3 joints
Links:
- link wl_link: geometry collision mesh filename=package://puzzlebot_localisation/models/MCR2_1000_1_1_Wheel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; visual mesh filename=package://puzzlebot_localisation/models/MCR2_1000_1_1_Wheel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
- link wr_link: geometry collision mesh filename=package://puzzlebot_localisation/models/MCR2_1000_1_1_Wheel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; visual mesh filename=package://puzzlebot_localisation/models/MCR2_1000_1_1_Wheel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
Joints:
- joint leftWheel: axis (none) -> 1 0 0
- joint rightWheel: axis (none) -> 1 0 0

Commit message: feat: :sparkles: Added new steps for getting wheel rotation

File: urdf/puzzlebot_jetson_ed_urdf.urdf (robot description, URDF)
Before this commit: robot Puzzlebot Jetson-Lidar Ed., 4 links, 3 joints
Joints:
- joint leftWheel: axis 1 0 0 -> 0 1 0
- joint rightWheel: axis 1 0 0 -> 0 1 0

Commit message: fix: :bug: Changed urdf model for having wheels rotating properly

File: urdf/puzzlebot_jetson_ed_urdf.urdf (robot description, URDF)
Before this commit: robot Puzzlebot Jetson-Lidar Ed., 4 links, 3 joints
Joints:
- joint leftWheel: axis 0 1 0 -> 0 0 1; origin xyz=0.0 0.0 0.0 -> xyz=0.05 -0.095 0 rpy=-1.57079632679 0 0
- joint rightWheel: axis 0 1 0 -> 0 0 1; origin xyz=0.0 0.0 0.0 -> xyz=0.05 0.095 0 rpy=1.57079632679 0 0
